File: trafficlight.sch (KiCad schematic (older format))
At the start: 7 parts, among them P1 CONN_6

Commit message: Added pin labelling on schematic, for use with Arduino.
Other:
- note added: "Arduino\npin numbers"
- note added: "D10"
- note added: "D11"
- note added: "D12"
- note added: "D13"
- note added: "D9"
- note added: "GND"
Changed lines of the file:
@@
 LIBS:contrib
 LIBS:valves
+LIBS:trafficlight-cache
 EELAYER 27 0
 EELAYER END
@@
 Sheet 1 1
 Title ""
-Date "19 jul 2015"
+Date "2 aug 2015"
 Rev ""
 Comp ""
@@
 Text Label 3550 3050 0    60   ~ 0
 GREEN
+Text Notes 2850 3600 0    60   ~ 0
+GND
+Text Notes 2850 3500 0    60   ~ 0
+D13
+Text Notes 2850 3400 0    60   ~ 0
+D12
+Text Notes 2850 3200 0    60   ~ 0
+D10
+Text Notes 2850 3300 0    60   ~ 0
+D11
+Text Notes 2850 3100 0    60   ~ 0
+D9
+Text Notes 2250 3300 0    60   ~ 0
+Arduino\npin numbers
 $EndSCHEMATC
