File: trafficlight.sch (KiCad schematic (older format))
At the start: 7 parts, among them P1 CONN_6

Commit message: Update to KiCad V4.0.4 as intermediate step.
Beware: the LEDs seem to have been reversed, pin 1/2 swap. But the PCB still shows pin 1 as the positive terminal, connected to the resistor. Will need to fix that once we've updated all the way to the latest version.
Parts:
- removed P1: CONN_6, symbol CONN_6
- added P1: CONN_01X06, symbol CONN_01X06
Changed lines of the file:
@@
 LIBS:memory
 LIBS:xilinx
-LIBS:special
 LIBS:microcontrollers
 LIBS:dsp
@@
 LIBS:valves
 LIBS:trafficlight-cache
-EELAYER 27 0
+EELAYER 25 0
 EELAYER END
 $Descr A4 11693 8268
@@
 Sheet 1 1
 Title "Traffic Signal Head for Arduino"
-Date "2 aug 2015"
-Rev "1.01"
-Comp ""
+Date "2024-10-13"
+Rev "1.02"
+Comp "John Honniball"
 Comment1 ""
 Comment2 ""
@@
 F 3 "~" H 4900 2900 60  0000 C CNN
 	1    4900 2900
-	1    0    0    -1
+	-1   0    0    1
 $EndComp
 $Comp
@@
 F 3 "~" H 4900 3300 60  0000 C CNN
 	1    4900 3300
-	1    0    0    -1
+	-1   0    0    1
 $EndComp
 $Comp
@@
 F 3 "~" H 4900 3700 60  0000 C CNN
 	1    4900 3700
-	1    0    0    -1
-$EndComp
-$Comp
-L CONN_6 P1
-U 1 1 55AB6F2B
-P 3150 3300
-F 0 "P1" V 3100 3300 60  0000 C CNN
-F 1 "CONN_6" V 3200 3300 60  0000 C CNN
-F 2 "" H 3150 3300 60  0000 C CNN
-F 3 "" H 3150 3300 60  0000 C CNN
-	1    3150 3300
 	-1   0    0    1
 $EndComp
@@
 $EndComp
 Wire Wire Line
-	5100 2900 5150 2900
-Wire Wire Line
 	5150 2900 5150 4050
-Wire Wire Line
-	5100 3300 5150 3300
 Connection ~ 5150 3300
-Wire Wire Line
-	5100 3700 5150 3700
 Connection ~ 5150 3700
-Wire Wire Line
-	4550 3700 4700 3700
-Wire Wire Line
-	4550 3300 4700 3300
-Wire Wire Line
-	4550 2900 4700 2900
 Wire Wire Line
 	3500 3550 3600 3550
@@
 	3900 3050 3900 2900
 Wire Wire Line
-	3900 2900 4050 2900
+	3900 2900 4150 2900
 Wire Wire Line
 	3500 3150 3900 3150
@@
 	3900 3150 3900 3300
 Wire Wire Line
-	3900 3300 4050 3300
+	3900 3300 4150 3300
 Wire Wire Line
 	3500 3250 3800 3250
@@
 	3800 3250 3800 3700
 Wire Wire Line
-	3800 3700 4050 3700
+	3800 3700 4150 3700
 Text Label 3550 3250 0    60   ~ 0
 RED
@@
 Text Notes 2250 3300 0    60   ~ 0
 Arduino\npin numbers
+$Comp
+L CONN_01X06 P1
+U 1 1 670C2FCB
+P 3300 3300
+F 0 "P1" H 3300 3650 50  0000 C CNN
+F 1 "CONN_01X06" V 3400 3300 50  0000 C CNN
+F 2 "" H 3300 3300 50  0000 C CNN
+F 3 "" H 3300 3300 50  0000 C CNN
+	1    3300 3300
+	-1   0    0    1
+$EndComp
+Wire Wire Line
+	4450 2900 4700 2900
+Wire Wire Line
+	4450 3300 4700 3300
+Wire Wire Line
+	4450 3700 4700 3700
+Wire Wire Line
+	5100 2900 5150 2900
+Wire Wire Line
+	5100 3300 5150 3300
+Wire Wire Line
+	5100 3700 5150 3700
 $EndSCHEMATC

Commit message: Update to KiCad V5.1.5 as intermediate step.
We're aiming for V8.0 but have to go via 4, 5, and 6.
Parts:
- removed P1: CONN_01X06, symbol CONN_01X06
- added P1: Conn_01x06, Connector_PinHeader_2.54mm:PinHeader_1x06_P2.54mm_Horizontal, symbol Connector_Generic:Conn_01x06
- D1, D2, D3: footprint ~ -> LED_THT:LED_D10.0mm; symbol LED -> Device:LED
- R1, R2, R3: footprint ~ -> Resistor_THT:R_Axial_DIN0204_L3.6mm_D1.6mm_P7.62mm_Horizontal; symbol R -> Device:R
Connections:
- wire segments 19 -> 22
Changed lines of the file:
@@
-EESchema Schematic File Version 2
-LIBS:power
-LIBS:device
-LIBS:transistors
-LIBS:conn
-LIBS:linear
-LIBS:regul
-LIBS:74xx
-LIBS:cmos4000
-LIBS:adc-dac
-LIBS:memory
-LIBS:xilinx
-LIBS:microcontrollers
-LIBS:dsp
-LIBS:microchip
-LIBS:analog_switches
-LIBS:motorola
-LIBS:texas
-LIBS:intel
-LIBS:audio
-LIBS:interface
-LIBS:digital-audio
-LIBS:philips
-LIBS:display
-LIBS:cypress
-LIBS:siliconi
-LIBS:opto
-LIBS:atmel
-LIBS:contrib
-LIBS:valves
-LIBS:trafficlight-cache
-EELAYER 25 0
+EESchema Schematic File Version 4
+EELAYER 30 0
 EELAYER END
 $Descr A4 11693 8268
@@
 $EndDescr
 $Comp
-L R R1
+L Device:R R1
 U 1 1 55AB6E54
 P 4300 2900
 F 0 "R1" V 4380 2900 40  0000 C CNN
 F 1 "330R" V 4307 2901 40  0000 C CNN
-F 2 "~" V 4230 2900 30  0000 C CNN
+F 2 "Resistor_THT:R_Axial_DIN0204_L3.6mm_D1.6mm_P7.62mm_Horizontal" V 4230 2900 30  0000 C CNN
 F 3 "~" H 4300 2900 30  0000 C CNN
 	1    4300 2900
@@
 $EndComp
 $Comp
-L R R2
+L Device:R R2
 U 1 1 55AB6E63
 P 4300 3300
 F 0 "R2" V 4380 3300 40  0000 C CNN
 F 1 "330R" V 4307 3301 40  0000 C CNN
-F 2 "~" V 4230 3300 30  0000 C CNN
+F 2 "Resistor_THT:R_Axial_DIN0204_L3.6mm_D1.6mm_P7.62mm_Horizontal" V 4230 3300 30  0000 C CNN
 F 3 "~" H 4300 3300 30  0000 C CNN
 	1    4300 3300
@@
 $EndComp
 $Comp
-L R R3
+L Device:R R3
 U 1 1 55AB6E72
 P 4300 3700
 F 0 "R3" V 4380 3700 40  0000 C CNN
 F 1 "330R" V 4307 3701 40  0000 C CNN
-F 2 "~" V 4230 3700 30  0000 C CNN
+F 2 "Resistor_THT:R_Axial_DIN0204_L3.6mm_D1.6mm_P7.62mm_Horizontal" V 4230 3700 30  0000 C CNN
 F 3 "~" H 4300 3700 30  0000 C CNN
 	1    4300 3700
@@
 $EndComp
 $Comp
-L LED D1
+L Device:LED D1
 U 1 1 55AB6EFE
 P 4900 2900
 F 0 "D1" H 4900 3000 50  0000 C CNN
 F 1 "Green LED" H 4900 2800 50  0000 C CNN
-F 2 "~" H 4900 2900 60  0000 C CNN
+F 2 "LED_THT:LED_D10.0mm" H 4900 2900 60  0000 C CNN
 F 3 "~" H 4900 2900 60  0000 C CNN
 	1    4900 2900
@@
 $EndComp
 $Comp
-L LED D2
+L Device:LED D2
 U 1 1 55AB6F0D
 P 4900 3300
 F 0 "D2" H 4900 3400 50  0000 C CNN
 F 1 "Amber LED" H 4900 3200 50  0000 C CNN
-F 2 "~" H 4900 3300 60  0000 C CNN
+F 2 "LED_THT:LED_D10.0mm" H 4900 3300 60  0000 C CNN
 F 3 "~" H 4900 3300 60  0000 C CNN
 	1    4900 3300
@@
 $EndComp
 $Comp
-L LED D3
+L Device:LED D3
 U 1 1 55AB6F1C
 P 4900 3700
 F 0 "D3" H 4900 3800 50  0000 C CNN
 F 1 "Red LED" H 4900 3600 50  0000 C CNN
-F 2 "~" H 4900 3700 60  0000 C CNN
+F 2 "LED_THT:LED_D10.0mm" H 4900 3700 60  0000 C CNN
 F 3 "~" H 4900 3700 60  0000 C CNN
 	1    4900 3700
@@
 $EndComp
 $Comp
-L GND #PWR01
+L power:GND #PWR01
 U 1 1 55AB6F5B
 P 5150 4050
@@
 	1    0    0    -1
 $EndComp
-Wire Wire Line
-	5150 2900 5150 4050
-Connection ~ 5150 3300
-Connection ~ 5150 3700
 Wire Wire Line
 	3500 3550 3600 3550
@@
 Text Notes 2250 3300 0    60   ~ 0
 Arduino\npin numbers
+Wire Wire Line
+	5150 3900 5150 4050
 $Comp
-L CONN_01X06 P1
-U 1 1 670C2FCB
-P 3300 3300
-F 0 "P1" H 3300 3650 50  0000 C CNN
-F 1 "CONN_01X06" V 3400 3300 50  0000 C CNN
-F 2 "" H 3300 3300 50  0000 C CNN
-F 3 "" H 3300 3300 50  0000 C CNN
-	1    3300 3300
+L Connector_Generic:Conn_01x06 P1
+U 1 1 6713FCA8
+P 3300 3350
+F 0 "P1" H 3218 2825 50  0000 C CNN
+F 1 "Conn_01x06" H 3218 2916 50  0000 C CNN
+F 2 "Connector_PinHeader_2.54mm:PinHeader_1x06_P2.54mm_Horizontal" H 3300 3350 50  0001 C CNN
+F 3 "~" H 3300 3350 50  0001 C CNN
+	1    3300 3350
 	-1   0    0    1
 $EndComp
 Wire Wire Line
-	4450 2900 4700 2900
+	5150 2900 5150 3300
 Wire Wire Line
-	4450 3300 4700 3300
+	4450 3300 4750 3300
 Wire Wire Line
-	4450 3700 4700 3700
+	4450 3700 4750 3700
 Wire Wire Line
-	5100 2900 5150 2900
+	5050 3700 5150 3700
+Connection ~ 5150 3700
 Wire Wire Line
-	5100 3300 5150 3300
+	5150 3700 5150 3900
 Wire Wire Line
-	5100 3700 5150 3700
+	5050 3300 5150 3300
+Connection ~ 5150 3300
+Wire Wire Line
+	5150 3300 5150 3700
+Wire Wire Line
+	5050 2900 5150 2900
+Wire Wire Line
+	4450 2900 4750 2900
 $EndSCHEMATC
